Commit message: robot_v3_description: geometría visual fiel al robot real sin cambiar la cinemática
Geometría visual medida sobre el escaneo métrico de v2 (config/visual_v3.yaml,
tools/measure_v2_scan.py):
- Chasis de perfiles en dos niveles con esquinas achaflanadas, montantes, placa
  inferior, traviesas, electrónica y placa del Hokuyo.
- Columna como módulo lineal (guías, husillo, placas) y carro móvil con el elevador.
- Bandeja, carcasa y monitor inclinado 12.8° con pantalla.
- Ruedas con llanta y radio marcador; ruedas locas con horquilla.
- Cabezal con servos, soporte y micrófono; D435 con dimensiones y lentes de Intel.
- Piper con la malla visual oficial a color, simplificada (p95 < 1 mm).

Un DAE por link (meshes/structure) porque RViz2 aplica el material de la
primera visual a todo el link. Colisiones, inercias, joints, límites y frames
sin cambios; screen_link pasa al centro del monitor real (frame fijo, solo visual).

Otros:
- display.launch.py: arm_pose:=home|zero (por defecto la pose de reposo).
- gazebo.launch.py: spawners encadenados con --switch-timeout 60.
- Sin range() en xacro (avisos por stderr hacían abortar launch).
- validate_v3.py: falla ante stderr de xacro; DAE visuales = primitivas.
- Evidencias: 5 vistas v3/v2/superpuestas, diagnóstico de 'No Image'.

Co-Authored-By: Claude Opus 5.5 <noreply@anthropic.com>
Claude-Session: https://claude.ai/code/session_01HwH2ygx4nYLrvzNwgb2nKW

File: robot_v3_description/urdf/base.xacro (robot description, xacro)
@@ -6,6 +6,13 @@
     <xacro:property name="W" value="${B['wheels']}"/>
     <link name="base_footprint"/>
-    <xacro:box_link name="base_link" size="${B['chassis_box']['size']}" center="${B['chassis_box']['center']}"
-                    material="chassis_blue" mass="${S['masses_kg']['base_link']}"/>
+    <!-- Chasis: visual = estructura de perfiles en dos niveles (config/visual_v3.yaml); colisión = caja medida -->
+    <link name="base_link">
+      <xacro:visual_parts group="chassis"/>
+      <collision>
+        <origin xyz="${xyz_str(B['chassis_box']['center'])}" rpy="0 0 0"/>
+        <geometry><box size="${xyz_str(B['chassis_box']['size'])}"/></geometry>
+      </collision>
+      <xacro:box_inertial m="${S['masses_kg']['base_link']}" size="${B['chassis_box']['size']}" xyz="${xyz_str(B['chassis_box']['center'])}"/>
+    </link>
     <joint name="base_joint" type="fixed">
       <parent link="base_footprint"/>
@@ -16,9 +23,5 @@
     <xacro:macro name="drive_wheel" params="side">
       <link name="${side}_wheel">
-        <visual>
-          <origin xyz="0 0 0" rpy="${pi/2} 0 0"/>
-          <geometry><cylinder radius="${W['visual_radius']}" length="${W['width']}"/></geometry>
-          <material name="wheel_black"/>
-        </visual>
+        <xacro:visual_parts group="wheel"/>
         <collision>
           <origin xyz="0 0 0" rpy="${pi/2} 0 0"/>
@@ -39,8 +42,5 @@
     <xacro:macro name="rear_caster" params="side">
       <link name="rear_${side}_caster">
-        <visual>
-          <geometry><sphere radius="${B['casters']['radius']}"/></geometry>
-          <material name="caster_gray"/>
-        </visual>
+        <xacro:visual_parts group="caster"/>
         <collision>
           <geometry><sphere radius="${B['casters']['radius']}"/></geometry>
@@ -59,9 +59,5 @@
     <xacro:property name="Ls" value="${G['laser']}"/>
     <link name="laser_mount">
-      <visual>
-        <origin xyz="0 0 ${Ls['body_size'][2]/2}" rpy="0 0 0"/>
-        <geometry><box size="${xyz_str(Ls['body_size'])}"/></geometry>
-        <material name="hokuyo_dark"/>
-      </visual>
+      <xacro:visual_parts group="hokuyo"/>
       <collision>
         <origin xyz="0 0 ${Ls['body_size'][2]/2}" rpy="0 0 0"/>

File: robot_v3_description/urdf/common.xacro (robot description, xacro)
@@ -8,15 +8,13 @@
   <!-- Lista [x, y, z] -> "x y z" -->
   <xacro:property name="xyz_str" value="${lambda v: ' '.join(str(float(c)) for c in v)}"/>
-  <material name="chassis_blue"><color rgba="0.15 0.45 0.85 1.0"/></material>
-  <material name="wheel_black"><color rgba="0.10 0.10 0.10 1.0"/></material>
-  <material name="caster_gray"><color rgba="0.35 0.35 0.35 1.0"/></material>
-  <material name="column_aluminum"><color rgba="0.65 0.65 0.70 1.0"/></material>
-  <material name="cube_metallic"><color rgba="0.28 0.30 0.35 1.0"/></material>
-  <material name="screen_black"><color rgba="0.06 0.07 0.09 1.0"/></material>
-  <material name="pantilt_dark"><color rgba="0.18 0.18 0.18 1.0"/></material>
-  <material name="hokuyo_dark"><color rgba="0.12 0.12 0.12 1.0"/></material>
-  <material name="realsense_aluminum"><color rgba="0.75 0.75 0.75 1.0"/></material>
-  <material name="piper_gray"><color rgba="0.75 0.78 0.88 1.0"/></material>
   <material name="orbbec_black"><color rgba="0.08 0.08 0.08 1.0"/></material>
+  <!-- Geometría visual de la estructura: un DAE por link (meshes/structure/<grupo>.dae), generado desde las primitivas
+       de config/visual_v3.yaml con tools/make_structure_visuals.py. Un único <visual> por link porque RViz2 aplica el
+       material de la primera <visual> a todas las del link. Los colores van dentro del DAE. -->
+  <xacro:macro name="visual_parts" params="group">
+    <visual>
+      <geometry><mesh filename="${pkg}/meshes/structure/${group}.dae"/></geometry>
+    </visual>
+  </xacro:macro>
   <!-- Inercias de sólidos homogéneos (masa provisional de config/sim_provisional.yaml) -->
   <xacro:macro name="box_inertial" params="m size xyz:='0 0 0'">
@@ -43,18 +41,3 @@
     </inertial>
   </xacro:macro>
-  <!-- Link con una caja como visual y colisión -->
-  <xacro:macro name="box_link" params="name size center material mass">
-    <link name="${name}">
-      <visual>
-        <origin xyz="${xyz_str(center)}" rpy="0 0 0"/>
-        <geometry><box size="${xyz_str(size)}"/></geometry>
-        <material name="${material}"/>
-      </visual>
-      <collision>
-        <origin xyz="${xyz_str(center)}" rpy="0 0 0"/>
-        <geometry><box size="${xyz_str(size)}"/></geometry>
-      </collision>
-      <xacro:box_inertial m="${mass}" size="${size}" xyz="${xyz_str(center)}"/>
-    </link>
-  </xacro:macro>
 </robot>

File: robot_v3_description/urdf/head.xacro (robot description, xacro)
@@ -5,6 +5,5 @@
   mount = lift:   colgado de torso_lift_link (árbol de base_athome); misma pose con el elevador en cero.
   Ejes: pan sobre +Z, tilt sobre +Y (positivo = cámara hacia abajo), como en base_athome.
-  Las piezas visuales son prismas simples del tamaño de un XL430 (28.5 x 34 x 46.5 mm, hoja de datos);
-  las posiciones de los ejes son las de config/geometry_v3.yaml (head).
+  Piezas visuales: config/visual_v3.yaml (servos XL430, soporte, micrófono); ejes: config/geometry_v3.yaml (head).
 -->
 <robot xmlns:xacro="http://www.ros.org/wiki/xacro">
@@ -15,9 +14,5 @@
     </xacro:if>
     <link name="pan_tilt_base_link">
-      <visual>
-        <origin xyz="0 0 0.003" rpy="0 0 0"/>
-        <geometry><box size="0.06 0.06 0.006"/></geometry>
-        <material name="pantilt_dark"/>
-      </visual>
+      <xacro:visual_parts group="pan_tilt_base"/>
       <xacro:box_inertial m="${S['masses_kg']['pan_tilt_base_link']}" size="${[0.06, 0.06, 0.006]}" xyz="0 0 0.003"/>
     </link>
@@ -30,9 +25,5 @@
     <xacro:property name="hz" value="${H['tilt_axis_above_pan']}"/>
     <link name="pan_link">
-      <visual>
-        <origin xyz="0 0 ${hz/2}" rpy="0 0 0"/>
-        <geometry><box size="0.034 0.0285 ${hz}"/></geometry>
-        <material name="pantilt_dark"/>
-      </visual>
+      <xacro:visual_parts group="pan"/>
       <collision>
         <origin xyz="0 0 ${hz/2}" rpy="0 0 0"/>
@@ -51,9 +42,5 @@
     <!-- Soporte de tilt: une el eje de tilt con la cámara -->
     <link name="tilt_link">
-      <visual>
-        <origin xyz="0.012 0 0" rpy="0 0 0"/>
-        <geometry><box size="0.024 0.050 0.010"/></geometry>
-        <material name="pantilt_dark"/>
-      </visual>
+      <xacro:visual_parts group="tilt"/>
       <xacro:box_inertial m="${S['masses_kg']['tilt_link']}" size="${[0.024, 0.05, 0.01]}" xyz="0.012 0 0"/>
     </link>

File: robot_v3_description/urdf/piper.xacro (robot description, xacro)
@@ -11,5 +11,6 @@
     * se elimina el link "world"; el brazo cuelga de "parent" con el origen recibido.
     * límites según el perfil "limits" de config/piper_limits.yaml.
-    * visual: mallas simplificadas (meshes/piper/visual, tools/simplify_piper_meshes.py); colisión: oficiales.
+    * visual: mallas visuales oficiales (DAE con colores) simplificadas, desvío p95 < 1 mm
+      (meshes/piper/visual, tools/make_piper_visuals.py); colisión: STL oficiales sin cambios.
     * tcp_link y cámara de muñeca (arm_camera_link) como en base_athome.
 -->
@@ -24,6 +25,6 @@
       <visual>
         <origin xyz="0 0 0" rpy="0 0 0"/>
-        <geometry><mesh filename="${pkg}/meshes/piper/visual/${'base_link' if name == 'arm_base_link' else name}.stl"/></geometry>
-        <material name="piper_gray"/>
+        <!-- DAE con los colores oficiales (blanco, negro, rojo); sin material para no sobrescribirlos -->
+        <geometry><mesh filename="${pkg}/meshes/piper/visual/${'base_link' if name == 'arm_base_link' else name}.dae"/></geometry>
       </visual>
       <collision>

File: robot_v3_description/urdf/realsense_d435.xacro (robot description, xacro)
@@ -37,9 +37,5 @@
     </joint>
     <link name="${name}_link">
-      <visual>
-        <origin xyz="0 ${-D['depth_py']} 0" rpy="0 0 0"/>
-        <geometry><box size="${D['cam_depth']} ${D['cam_width']} ${D['cam_height']}"/></geometry>
-        <material name="realsense_aluminum"/>
-      </visual>
+      <xacro:visual_parts group="d435"/>
       <collision>
         <origin xyz="0 ${-D['depth_py']} 0" rpy="0 0 0"/>

File: robot_v3_description/urdf/torso.xacro (robot description, xacro)
@@ -11,6 +11,13 @@
     <xacro:property name="SL" value="${S['lift']}"/>
     <!-- Nombres de base_athome (torso_column, torso_lift_link, mounting_cube_link, screen_link) -->
-    <xacro:box_link name="torso_column" size="${T['column']['box_size']}" center="${T['column']['box_center']}"
-                    material="column_aluminum" mass="${S['masses_kg']['torso_column']}"/>
+    <!-- Columna: módulo lineal (paredes, guías, husillo, placas); colisión = caja medida -->
+    <link name="torso_column">
+      <xacro:visual_parts group="column"/>
+      <collision>
+        <origin xyz="${xyz_str(T['column']['box_center'])}" rpy="0 0 0"/>
+        <geometry><box size="${xyz_str(T['column']['box_size'])}"/></geometry>
+      </collision>
+      <xacro:box_inertial m="${S['masses_kg']['torso_column']}" size="${T['column']['box_size']}" xyz="${xyz_str(T['column']['box_center'])}"/>
+    </link>
     <joint name="torso_column_joint" type="fixed">
       <parent link="base_link"/>
@@ -20,4 +27,5 @@
     <!-- Carro del elevador: referencia del movimiento, sobre el eje de la columna -->
     <link name="torso_lift_link">
+      <xacro:visual_parts group="carriage"/>
       <xacro:box_inertial m="${S['masses_kg']['torso_lift_link']}" size="${[0.05, 0.05, 0.05]}"/>
     </link>
@@ -30,6 +38,12 @@
     </joint>
     <!-- Caja superior (bandeja + monitor + carro), dimensiones medidas -->
-    <xacro:box_link name="mounting_cube_link" size="${T['box']['size']}" center="${[0, 0, 0]}"
-                    material="cube_metallic" mass="${S['masses_kg']['mounting_cube_link']}"/>
+    <!-- Bandeja + carcasa + monitor inclinado (visual); colisión = caja envolvente medida -->
+    <link name="mounting_cube_link">
+      <xacro:visual_parts group="upper_box"/>
+      <collision>
+        <geometry><box size="${xyz_str(T['box']['size'])}"/></geometry>
+      </collision>
+      <xacro:box_inertial m="${S['masses_kg']['mounting_cube_link']}" size="${T['box']['size']}"/>
+    </link>
     <joint name="torso_lift_to_cube_joint" type="fixed">
       <parent link="torso_lift_link"/>
@@ -37,18 +51,14 @@
       <origin xyz="${xyz_str(T['box']['center_in_lift'])}" rpy="0 0 0"/>
     </joint>
-    <!-- Pantalla HRI en la cara frontal de la caja (solo visual, 1 cm por delante de la caja medida para que se vea; su colisión está incluida en la caja) -->
+    <!-- Pantalla HRI: frame en el centro de la cara frontal del monitor (x = normal hacia afuera), inclinado como en el escaneo.
+         Solo visual; su colisión está incluida en la caja. -->
     <link name="screen_link">
-      <visual>
-        <origin xyz="${T['screen']['size'][0]/2} 0 0" rpy="0 0 0"/>
-        <geometry><box size="${xyz_str(T['screen']['size'])}"/></geometry>
-        <material name="screen_black"/>
-      </visual>
-      <xacro:box_inertial m="${S['masses_kg']['screen_link']}" size="${T['screen']['size']}"
-                          xyz="${T['screen']['size'][0]/2} 0 0"/>
+      <xacro:visual_parts group="screen"/>
+      <xacro:box_inertial m="${S['masses_kg']['screen_link']}" size="${T['screen']['size']}"/>
     </link>
     <joint name="torso_lift_to_screen_joint" type="fixed">
       <parent link="mounting_cube_link"/>
       <child link="screen_link"/>
-      <origin xyz="${xyz_str(T['screen']['center_in_box'])}" rpy="0 0 0"/>
+      <origin xyz="${xyz_str(T['screen']['center_in_box'])}" rpy="${xyz_str(T['screen']['rpy'])}"/>
     </joint>
   </xacro:macro>
