Commit message: robot_v3_description: pinza del Piper con un solo grado de libertad (joint8 mimic de joint7)
- joint8 = -1 · joint7 (<mimic>), relación oficial de AgileX (agx_arm_urdf:
  dedos = ±0.5·gripper); mismos orígenes, ejes, límites y geometría.
- joint_state_publisher_gui muestra un solo slider de pinza (joint7).
- ros2_control: joint8 sin interfaz de comando, declarado mimic (Humble por
  parámetros, Jazzy por el URDF); gripper_controller comanda solo joint7.
- Compatibilidad con la Jetson: joint7/joint8 publicados siguen siendo válidos.
- demo_motion, runtime_checks, check_real_state y validate_v3 adaptados; pinza
  cerrada, a mitad y abierta verificada.
- Validado en Humble (estático 69/69, mock 26/26, Gazebo 32/32, real_state 9/9)
  y Jazzy (estático 69/69, mock 26/26, real_state 9/9, GUI con 12 sliders).

Co-Authored-By: Claude Opus 5.5 <noreply@anthropic.com>
Claude-Session: https://claude.ai/code/session_01HwH2ygx4nYLrvzNwgb2nKW

File: robot_v3_description/urdf/piper.xacro (robot description, xacro)
@@ -95,6 +95,17 @@
     <xacro:piper_joint name="joint7" type="prismatic" parent="gripper_base" child="link7"
                        xyz="0 0 0.1358" rpy="1.5707963 0 0" lim="${LG['joint7']}"/>
-    <xacro:piper_joint name="joint8" type="prismatic" parent="gripper_base" child="link8"
-                       xyz="0 0 0.1358" rpy="1.5707963 0 -3.1415926" lim="${LG['joint8']}" axis="0 0 -1"/>
+    <!-- La pinza tiene UN grado de libertad: joint7 es la apertura de cada dedo y joint8 la copia con signo opuesto.
+         Relación oficial de AgileX (agx_arm_urdf, piper_with_gripper_description.xacro): dedo1 = +0.5·gripper,
+         dedo2 = -0.5·gripper, con los mismos orígenes, ejes y mallas que joint7/joint8 -> joint8 = -1 · joint7.
+         Coincide con lo que publica la Jetson: joint7 = +apertura/2, joint8 = -apertura/2. -->
+    <joint name="joint8" type="prismatic">
+      <origin xyz="0 0 0.1358" rpy="1.5707963 0 -3.1415926"/>
+      <parent link="gripper_base"/>
+      <child link="link8"/>
+      <axis xyz="0 0 -1"/>
+      <limit lower="${LG['joint8']['lower']}" upper="${LG['joint8']['upper']}" effort="${LG['joint8']['effort']}"
+             velocity="${LG['joint8']['velocity']}"/>
+      <mimic joint="joint7" multiplier="${LG['joint8']['mimic_multiplier']}" offset="0"/>
+    </joint>
     <!-- Punto central de herramienta entre los dedos (base_athome / piper_ros) -->
     <link name="tcp_link"/>

File: robot_v3_description/urdf/ros2_control.xacro (robot description, xacro)
@@ -43,5 +43,13 @@
       <xacro:position_joint name="joint6"/>
       <xacro:position_joint name="joint7"/>
-      <xacro:position_joint name="joint8"/>
+      <!-- joint8 = -1 · joint7 (mimic en el URDF). Sin interfaz de comando: la pinza tiene una sola orden lógica.
+           Humble (ros2_control 2.x, mock e ign_ros2_control) toma la relación de estos parámetros;
+           Jazzy (4.x) la toma del <mimic> del URDF. -->
+      <joint name="joint8">
+        <param name="mimic">joint7</param>
+        <param name="multiplier">-1</param>
+        <state_interface name="position"/>
+        <state_interface name="velocity"/>
+      </joint>
       <xacro:position_joint name="pan_joint"/>
       <xacro:position_joint name="tilt_joint"/>
