Commit message: Agarre físico en Gazebo: precierre, descenso verificado, acoplamiento de dedos y entrenamiento headless
- Pinza: orden abierta = precierre a 32 mm (nunca 35), rampa de cierre, detección de dedos detenidos por el objeto
  (objetivo ordenado vs posición medida) y error de mimic en la observación del estado de tarea.
- Experto: orientación con eje de cierre perpendicular a las caras del cubo y descenso planificado/verificado
  (waypoints < 2 mm, < 3°); apriete y levantamiento con escalado uniforme. Se conservan los cambios de 8224a69.
- Simulación: gripper_servo:=dual (joint8 con servo propio, mimic=false solo en ros2_control gz) y ley de centrado
  a 50 Hz (solverbot_rl/gripper.py) que emula el acoplamiento rígido del Piper; corrige la deriva en bloque de los
  dedos medida en Gazebo. Cinemática y modo del robot real sin cambios.
- Backend: subpasos sincronizados por reloj, rclpy sin manejadores de señales, cierre limpio, verificación de
  sensores cuando la observación los usa.
- validate_grasp.py: validación física por semilla (CSV/JSON). Resultado: 20/20 semillas 40000-40019, cubo >= 30 mm
  sostenido 4 s, |j7+j8| <= 2 mm. validate_sim.py: TODO OK 3/3.
- train.py: checkpoints atómicos con replay buffer, reanudación automática, parada limpia por SIGTERM, progreso.
- tools/headless: setup, start/status/stop, orquestador y unidad systemd de usuario (probados en Cloud).
- 37 pruebas unitarias (12 nuevas de pinza/precierre/acoplamiento/descenso).

Co-Authored-By: Claude Opus 5.5 <noreply@anthropic.com>
Claude-Session: https://claude.ai/code/session_01Kcbwvy3KLEBhjvQeMfMCFy

File: robot_v3_description/urdf/robot_v3.urdf.xacro (robot description, xacro)
@@ -19,4 +19,5 @@
     camera_profile demo | train          resolución/frecuencia de las cámaras simuladas (config/sim_cameras.yaml)
     controllers   ruta a un YAML de ros2_control (por defecto config/ros2_controllers.yaml)
+    gripper_servo mimic | dual            dual: joint8 con servo propio y orden espejada (solo simulación, ver ros2_control.xacro)
 -->
 <robot name="robot_v3" xmlns:xacro="http://www.ros.org/wiki/xacro">
@@ -27,4 +28,5 @@
   <xacro:arg name="wrist_camera" default="true"/>
   <xacro:arg name="camera_profile" default="demo"/>
+  <xacro:arg name="gripper_servo" default="mimic"/>
   <xacro:arg name="controllers" default="$(find robot_v3_description)/config/ros2_controllers.yaml"/>
   <xacro:property name="ros2_control_mode" value="$(arg ros2_control)"/>
@@ -50,5 +52,5 @@
   <xacro:if value="${ros2_control_mode != 'none'}">
     <xacro:include filename="$(find robot_v3_description)/urdf/ros2_control.xacro"/>
-    <xacro:robot_v3_ros2_control mode="${ros2_control_mode}"/>
+    <xacro:robot_v3_ros2_control mode="${ros2_control_mode}" gripper_servo="$(arg gripper_servo)"/>
   </xacro:if>
   <xacro:if value="${ros2_control_mode == 'gazebo'}">

File: robot_v3_description/urdf/ros2_control.xacro (robot description, xacro)
@@ -16,5 +16,8 @@
     </joint>
   </xacro:macro>
-  <xacro:macro name="robot_v3_ros2_control" params="mode">
+  <xacro:macro name="robot_v3_ros2_control" params="mode gripper_servo:=mimic">
+    <xacro:if value="${gripper_servo not in ['mimic', 'dual'] or (gripper_servo == 'dual' and mode != 'gz')}">
+      ${xacro.fatal('gripper_servo: mimic | dual (dual solo con ros2_control:=gz); recibido ' + gripper_servo)}
+    </xacro:if>
     <ros2_control name="robot_v3_sim" type="system">
       <hardware>
@@ -50,10 +53,23 @@
            Humble (ros2_control 2.x, mock e ign_ros2_control) toma la relación de estos parámetros;
            Jazzy (4.x) la toma del <mimic> del URDF. -->
-      <joint name="joint8">
-        <param name="mimic">joint7</param>
-        <param name="multiplier">-1</param>
-        <state_interface name="position"/>
-        <state_interface name="velocity"/>
-      </joint>
+      <xacro:unless value="${gripper_servo == 'dual'}">
+        <joint name="joint8">
+          <param name="mimic">joint7</param>
+          <param name="multiplier">-1</param>
+          <state_interface name="position"/>
+          <state_interface name="velocity"/>
+        </joint>
+      </xacro:unless>
+      <!-- SOLO SIMULACIÓN (gz): el mimic emulado por gz_ros2_control no ejerce fuerza propia en joint8 y, al apretar un
+           objeto, el par de dedos se desplaza en bloque hasta el tope de joint8 (Gazebo, 2026-10-27). En el Piper real
+           ambos dedos están acoplados rígidamente a un solo motor; se emula con un servo de posición por dedo que
+           recibe la MISMA orden espejada (la pinza sigue teniendo una sola orden lógica en el entorno). -->
+      <xacro:if value="${gripper_servo == 'dual'}">
+        <joint name="joint8" mimic="false">
+          <command_interface name="position"/>
+          <state_interface name="position"/>
+          <state_interface name="velocity"/>
+        </joint>
+      </xacro:if>
       <xacro:position_joint name="pan_joint"/>
       <xacro:position_joint name="tilt_joint"/>
